File: Bald Sense Wing v1-before rough layout.kicad_pcb (KiCad board)
At the start: 4 copper layers, 50.8 x 22.9 mm, 43 parts, among them J1 feather long, J2 feather short, J3 1140084168, Q1 Q_PNP_BEC, Q2 Q_NPN_BEC, U1 APDS-9960, U2 DS3231MZ, U3 SHT30-DIS, U4 MIC5504-3.3YM5, U5 CMM-4737DT-26186-TR

Commit message: Minor updates
Parts:
- moved JP3 1.73 mm to (68.5, 36.6)
- moved R3 1.73 mm to (68.6, 36.8)
- moved R13 1.05 mm to (66.3, 30.0), turned to 0 degrees
- moved R12 1.00 mm to (70.8, 30.0), turned to 180 degrees
- moved C4 0.58 mm to (70.5, 36.7), turned to 90 degrees
- moved C1 0.58 mm to (70.5, 40.6), turned to 90 degrees
- moved C3 0.58 mm to (70.5, 33.0), turned to 90 degrees
Routing:
- net /SDA: track 2.77 -> 0.00 mm
- net /SCL: track 2.77 -> 0.00 mm
Other:
- copper layers 4 -> 2
- net class Default: via_dia 0.4064 -> 0.8; via_drill 0.3048 -> 0.4
