File: Bald Sense Wing v1.sch (KiCad schematic (older format))
At the start: 19 parts, among them J1 feather long, J2 feather short

Commit message: Inital PCB Footprint Placements
Thank you to everyone in the live stream chat.
Parts:
- added C5, C6: 1uF, Capacitor_SMD:C_0805_2012Metric, symbol Device:C_Small
- added D1: PWR_LED, LED_SMD:LED_1206_3216Metric, symbol Device:LED_Small_ALT
- added JP1, JP5: SolderJumper_2_Open, Jumper:SolderJumper-2_P1.3mm_Open_RoundedPad1.0x1.5mm, symbol Jumper:SolderJumper_2_Open
- added JP2: M02, Connector_PinSocket_2.54mm:PinSocket_1x02_P2.54mm_Vertical, symbol freetronics_schematic:M02
- added JP4: SolderJumper_2_Bridged, Jumper:SolderJumper-2_P1.3mm_Bridged_RoundedPad1.0x1.5mm, symbol Jumper:SolderJumper_2_Bridged
- added JP6: SolderJumper_3_Bridged12, Jumper:SolderJumper-3_P1.3mm_Bridged12_RoundedPad1.0x1.5mm, symbol Jumper:SolderJumper_3_Bridged12
- added Q1: Q_PNP_BEC, Package_TO_SOT_SMD:SOT-323_SC-70, symbol Device:Q_PNP_BEC
- added Q2: Q_NPN_BEC, Package_TO_SOT_SMD:SOT-23, symbol Device:Q_NPN_BEC
- added R10, R14, R7: 10K, Resistor_SMD:R_0805_2012Metric, symbol Device:R_Small
- added R11, R8, R9: 1K, Resistor_SMD:R_0805_2012Metric, symbol Device:R_Small
- added R4: DNP, Resistor_SMD:R_0805_2012Metric, symbol Device:R_Small
- added R5, R6: 4.7K, Resistor_SMD:R_0805_2012Metric, symbol Device:R_Small
- added U4: MIC5504-3.3YM5, Package_TO_SOT_SMD:SOT-23-5, symbol Regulator_Linear:MIC5504-3.3YM5
- J3: renamed from J?; footprint AMPHENOL_1140084168 -> My Libraries:AMPHENOL_1140084168; symbol My~Library:1140084168 -> My_Library:1140084168
- JP3: renamed from JP?; footprint (none) -> Jumper:SolderJumper-2_P1.3mm_Open_RoundedPad1.0x1.5mm
- MK1: renamed from MK?; footprint MIC_MP34DT01-M -> My Libraries:MIC_MP34DT01-M; symbol My~Library:MP34DT01-M -> My_Library:MP34DT01-M
- U1: renamed from U?; footprint APDS-9960 -> My Libraries:APDS-9960; symbol My~Library:APDS-9960 -> My_Library:APDS-9960
- U3: renamed from U?; footprint DFN250X250X100-9N -> My Libraries:DFN250X250X100-9N; symbol My~Library:SHT30-DIS -> My_Library:SHT30-DIS
- gave numbers to parts that had none: 12
Connections:
- net labels added: 3v3_Reg_En, 3v3_feather, Batt_Meas, Batt_Meas_En, RTC_BATT, SD-CD, SD-CS, VUSB_Meas
- net labels removed: A0, A1, A2, A3, A4, A5, F0, F1, F2, F3, F4, F5, F6, MISO, MOSI, SCK
- wire segments 118 -> 159
Other:
- note added: "LEDs are cool"
- note added: "On-board 3.3v regulator"
- note added: "Pads for I2C Pull-Up"
- note added: "TODO: Battery measuring circuit"
- note added: "USB Power Detection"
- note removed: "TODO: Header pin for 3.3v node, so we can test current usage"
- moved on the sheet: BT1, C1, C2, C3, C4, C7, J1, J2, JP3, R1, R12, R13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

Commit message: Re-arranged PCB
Moved SD Card slot to other side and put sensors on an edge.
Parts:
- JP1: value SolderJumper_2_Open -> 3.3V Select
- JP3: value SolderJumper_2_Open -> SHT30-Alert
- JP4: value SolderJumper_2_Bridged -> Reg En
- JP5: value SolderJumper_2_Open -> LED En
- JP6: value SolderJumper_3_Bridged12 -> RTC Batt Select
Changed lines of the file:
@@
 P 3350 3900
 F 0 "JP3" H 3350 4013 50  0000 C CNN
-F 1 "SolderJumper_2_Open" H 3350 4014 50  0001 C CNN
+F 1 "SHT30-Alert" H 3350 4014 50  0001 C CNN
 F 2 "Jumper:SolderJumper-2_P1.3mm_Open_RoundedPad1.0x1.5mm" H 3350 3900 50  0001 C CNN
 F 3 "~" H 3350 3900 50  0001 C CNN
@@
 	1    0    0    -1
 $EndComp
-Text Label 4050 3900 2    50   ~ 0
-SHT30-ALERT
 Wire Wire Line
 	3500 3900 4050 3900
@@
 P 9350 2900
 F 0 "JP1" H 9350 3013 50  0000 C CNN
-F 1 "SolderJumper_2_Open" H 9350 3014 50  0001 C CNN
+F 1 "3.3V Select" H 9350 3014 50  0001 C CNN
 F 2 "Jumper:SolderJumper-2_P1.3mm_Open_RoundedPad1.0x1.5mm" H 9350 2900 50  0001 C CNN
 F 3 "~" H 9350 2900 50  0001 C CNN
@@
 P 5900 5800
 F 0 "JP5" H 5900 5913 50  0000 C CNN
-F 1 "SolderJumper_2_Open" H 5900 5914 50  0001 C CNN
+F 1 "LED En" H 5900 5914 50  0001 C CNN
 F 2 "Jumper:SolderJumper-2_P1.3mm_Open_RoundedPad1.0x1.5mm" H 5900 5800 50  0001 C CNN
 F 3 "~" H 5900 5800 50  0001 C CNN
@@
 P 7500 4250
 F 0 "JP4" H 7500 4363 50  0000 C CNN
-F 1 "SolderJumper_2_Bridged" H 7500 4364 50  0001 C CNN
+F 1 "Reg En" H 7500 4364 50  0001 C CNN
 F 2 "Jumper:SolderJumper-2_P1.3mm_Bridged_RoundedPad1.0x1.5mm" H 7500 4250 50  0001 C CNN
 F 3 "~" H 7500 4250 50  0001 C CNN
@@
 P 3200 2350
 F 0 "JP6" H 3200 2463 50  0000 C CNN
-F 1 "SolderJumper_3_Bridged12" H 3200 2464 50  0001 C CNN
+F 1 "RTC Batt Select" H 3200 2464 50  0001 C CNN
 F 2 "Jumper:SolderJumper-3_P1.3mm_Bridged12_RoundedPad1.0x1.5mm" H 3200 2350 50  0001 C CNN
 F 3 "~" H 3200 2350 50  0001 C CNN
@@
 Wire Wire Line
 	3500 2350 3500 2300
+Text Label 4050 3900 2    50   ~ 0
+SHT30-ALERT
 $EndSCHEMATC

Commit message: Re-arranged PCB parts to a more logical layout
Switched to SOT-23 3906 because the SO70 looked too small.
Switched PDM to a Cui CMM-4737DT-26186.
Fixed two-pin header footprint (was socket before)
Changed to 10mm battery holder
Changed Footprint reference sizes
Parts:
- removed MK1: MP34DT01-M, My Libraries:MIC_MP34DT01-M, symbol My_Library:MP34DT01-M
- added U5: CMM-4737DT-26186-TR, My Libraries:XDCR_CMM-4737DT-26186-TR, symbol My_Library:CMM-4737DT-26186-TR
- BT1: value 12mm -> 10mm; footprint Battery:BatteryHolder_Keystone_3000_1x12mm -> My Libraries:MPD_BK-870
- JP2: footprint Connector_PinSocket_2.54mm:PinSocket_1x02_P2.54mm_Vertical -> Connector_PinHeader_2.54mm:PinHeader_1x02_P2.54mm_Vertical
- Q1: footprint Package_TO_SOT_SMD:SOT-323_SC-70 -> Package_TO_SOT_SMD:SOT-23; MPN MMBT3906WT1G -> MMBT3906LT3G; SPN 88H4789 -> 09R9450
Connections:
- net +3V3: now also U5.6 (VDD)
- net 32KHz: now also J2.7 (Pin_7); no longer J2.3 (Pin_3)
- net 3v3_Reg_En: now also J2.9 (Pin_9); no longer J1.12 (Pin_12)
- net Batt_Meas_En: now also J2.8 (Pin_8); no longer J1.11 (Pin_11)
- net DS3231_INT: now also J2.6 (Pin_6); no longer J2.4 (Pin_4)
- net GND: now also U5.1 (GND), U5.2 (L/R), U5.3 (GND)
- net PDM_CLK: now also J2.3 (Pin_3), U5.4 (CLOCK); no longer J2.7 (Pin_7)
- net PDM_DATA: now also J2.4 (Pin_4), U5.5 (DATA); no longer J2.6 (Pin_6)
- net SD-CD: now also J1.12 (Pin_12); no longer J2.9 (Pin_9)
- net SD-CS: now also J1.11 (Pin_11); no longer J2.8 (Pin_8)
Other:
- note added: "CMM-4737DT-26186 PDM MIC (Sound Sensor)"
- note removed: "MP34DT01TR-M PDM MIC (Sound Sensor)"
- note removed: "Note: What does the LR signal actually do?\nAnd what does CLK and Data look like on a scope?"
Changed lines of the file:
@@
 Text Label 8900 1150 0    50   ~ 0
 AREF
-Text Label 8800 1950 0    50   ~ 0
+Text Label 8550 1950 0    50   ~ 0
 SD_CLK
-Text Label 8800 2150 0    50   ~ 0
+Text Label 8550 2150 0    50   ~ 0
 SD_DOut
-Text Label 8800 2050 0    50   ~ 0
+Text Label 8550 2050 0    50   ~ 0
 SD_DIn
 Text Label 8900 2250 0    50   ~ 0
@@
 	8900 1150 9100 1150
 Wire Wire Line
-	8800 1950 9100 1950
-Wire Wire Line
-	8800 2150 9100 2150
+	8550 1950 9100 1950
+Wire Wire Line
+	8550 2150 9100 2150
 Wire Wire Line
 	8900 2250 9100 2250
@@
 P 700 1250
 F 0 "BT1" H 818 1346 50  0000 L CNN
-F 1 "12mm" H 818 1255 50  0000 L CNN
-F 2 "Battery:BatteryHolder_Keystone_3000_1x12mm" V 700 1310 50  0001 C CNN
+F 1 "10mm" H 818 1255 50  0000 L CNN
+F 2 "My Libraries:MPD_BK-870" V 700 1310 50  0001 C CNN
 F 3 "~" V 700 1310 50  0001 C CNN
 	1    700  1250
@@
 Text Notes 1550 750  0    50   ~ 0
 DS3231 RTC
-Wire Wire Line
-	6600 2250 6750 2250
-Connection ~ 6750 2250
-$Comp
-L power:GND #PWR0108
-U 1 1 5EC4ECD5
-P 6750 2300
-F 0 "#PWR0108" H 6750 2050 50  0001 C CNN
-F 1 "GND" H 6755 2127 50  0000 C CNN
-F 2 "" H 6750 2300 50  0001 C CNN
-F 3 "" H 6750 2300 50  0001 C CNN
-	1    6750 2300
-	1    0    0    -1
-$EndComp
-Wire Wire Line
-	6750 2300 6750 2250
 $Comp
 L power:+3.3V #PWR0109
 U 1 1 5EC50915
-P 7500 1200
-F 0 "#PWR0109" H 7500 1050 50  0001 C CNN
-F 1 "+3.3V" H 7515 1373 50  0000 C CNN
-F 2 "" H 7500 1200 50  0001 C CNN
-F 3 "" H 7500 1200 50  0001 C CNN
-	1    7500 1200
-	1    0    0    -1
-$EndComp
-Wire Wire Line
-	7500 1200 7500 1350
-Wire Wire Line
-	7500 1350 7400 1350
+P 8100 1150
+F 0 "#PWR0109" H 8100 1000 50  0001 C CNN
+F 1 "+3.3V" H 8115 1323 50  0000 C CNN
+F 2 "" H 8100 1150 50  0001 C CNN
+F 3 "" H 8100 1150 50  0001 C CNN
+	1    8100 1150
+	1    0    0    -1
+$EndComp
+Wire Wire Line
+	8100 1150 8100 1300
+Wire Wire Line
+	8100 1300 8000 1300
 $Comp
 L Device:C_Small C1
@@
 Wire Wire Line
 	6050 1000 6050 1050
-$Comp
-L power:GND #PWR0112
-U 1 1 5EC595AD
-P 6150 1800
-F 0 "#PWR0112" H 6150 1550 50  0001 C CNN
-F 1 "GND" H 6155 1627 50  0000 C CNN
-F 2 "" H 6150 1800 50  0001 C CNN
-F 3 "" H 6150 1800 50  0001 C CNN
-	1    6150 1800
-	1    0    0    -1
-$EndComp
-Wire Wire Line
-	6200 1750 6150 1750
-Wire Wire Line
-	6150 1750 6150 1800
-Wire Wire Line
-	6200 1600 5850 1600
-Text Label 5850 1600 0    50   ~ 0
-PDM_CLK
-Text Label 7800 1550 2    50   ~ 0
-PDM_DATA
-Wire Wire Line
-	7400 1550 7800 1550
 Text Notes 6600 900  0    50   ~ 0
-MP34DT01TR-M PDM MIC (Sound Sensor)
-Text Notes 6050 2750 0    50   ~ 0
-Note: What does the LR signal actually do?\nAnd what does CLK and Data look like on a scope?
+CMM-4737DT-26186 PDM MIC (Sound Sensor)
 Wire Wire Line
 	5200 1350 5350 1350
@@
 $EndComp
 $Comp
-L My_Library:MP34DT01-M MK1
-U 1 1 5ECFFEA3
-P 6800 1650
-F 0 "MK1" H 6800 2217 50  0000 C CNN
-F 1 "MP34DT01-M" H 6800 2126 50  0000 C CNN
-F 2 "My Libraries:MIC_MP34DT01-M" H 6150 600 50  0001 L BNN
-F 3 "" H 7000 850 50  0001 L BNN
-F 4 "MEMS audio sensor omnidirectional stereo digital microphone" H 5650 950 50  0001 L BNN "Field4"
-F 5 "None" H 7350 850 50  0001 L BNN "Field5"
-F 6 "Unavailable" H 6000 800 50  0001 L BNN "Field6"
-F 7 "STMicroelectronics" H 6150 700 50  0001 L BNN "Field7"
-F 8 "MP34DT01-M" H 7000 750 50  0001 L BNN "Field8"
-	1    6800 1650
-	1    0    0    -1
-$EndComp
-$Comp
 L Device:C_Small C7
 U 1 1 5ED0282F
@@
 Text Notes 8800 600  0    50   ~ 0
 TODO: Figure out pinout to feather board.\n(Pick two different feathers to make sure they "work.")
-Wire Wire Line
-	6750 2250 6900 2250
 Text Label 8650 1050 0    50   ~ 0
 3v3_feather
@@
 	6300 5800 6400 5800
 Wire Wire Line
-	8800 2050 9100 2050
-Text Label 10400 1650 2    50   ~ 0
+	8550 2050 9100 2050
+Text Label 8550 1350 0    50   ~ 0
 SD-CD
 $Comp
@@
 Wire Wire Line
 	3700 6000 3950 6000
-Text Label 10400 1750 2    50   ~ 0
+Text Label 8550 1450 0    50   ~ 0
 SD-CS
-Text Label 10400 1850 2    50   ~ 0
+Text Label 10400 2250 2    50   ~ 0
 PDM_CLK
-Text Label 10400 1950 2    50   ~ 0
+Text Label 10400 2150 2    50   ~ 0
 PDM_DATA
 Text Notes 8550 850  0    50   ~ 0
@@
 Text Label 10400 2050 2    50   ~ 0
 DS3231_RST
-Text Label 10400 2150 2    50   ~ 0
+Text Label 10400 1950 2    50   ~ 0
 DS3231_INT
-Text Label 10400 2250 2    50   ~ 0
+Text Label 10400 1850 2    50   ~ 0
 32KHz
 Text Label 8550 1850 0    50   ~ 0
@@
 Wire Wire Line
 	9250 5300 9400 5300
-Connection ~ 6900 2250
-Wire Wire Line
-	6900 2250 7050 2250
-Text Label 8550 1450 0    50   ~ 0
+Text Label 10400 1750 2    50   ~ 0
 Batt_Meas_En
 Wire Wire Line
@@
 F 0 "Q1" H 9991 5300 50  0000 L CNN
 F 1 "Q_PNP_BEC" H 9990 5345 50  0001 L CNN
-F 2 "Package_TO_SOT_SMD:SOT-323_SC-70" H 10000 5400 50  0001 C CNN
+F 2 "Package_TO_SOT_SMD:SOT-23" H 10000 5400 50  0001 C CNN
 F 3 "~" H 9800 5300 50  0001 C CNN
-F 4 "MMBT3906WT1G " H 9800 5300 50  0001 C CNN "MPN"
-F 5 "88H4789" H 9800 5300 50  0001 C CNN "SPN"
+F 4 "MMBT3906LT3G" H 9800 5300 50  0001 C CNN "MPN"
+F 5 "09R9450" H 9800 5300 50  0001 C CNN "SPN"
 F 6 "Newark" H 9800 5300 50  0001 C CNN "Supplier"
 	1    9800 5300
@@
 Text Label 5450 3600 3    50   ~ 0
 VBAT
-Text Label 8550 1350 0    50   ~ 0
+Text Label 10400 1650 2    50   ~ 0
 3v3_Reg_En
 Text Notes 6100 3400 0    50   ~ 0
@@
 F 0 "JP2" H 7728 3728 50  0000 L CNN
 F 1 "M02" H 7728 3644 40  0000 L CNN
-F 2 "Connector_PinSocket_2.54mm:PinSocket_1x02_P2.54mm_Vertical" H 7750 3750 60  0001 C CNN
+F 2 "Connector_PinHeader_2.54mm:PinHeader_1x02_P2.54mm_Vertical" H 7750 3750 60  0001 C CNN
 F 3 "" H 7750 3750 60  0000 C CNN
 	1    7750 3750
@@
 Text Label 4050 3900 2    50   ~ 0
 SHT30-ALERT
+$Comp
+L My_Library:CMM-4737DT-26186-TR U5
+U 1 1 5ECAD5C5
+P 7300 1600
+F 0 "U5" H 7300 2167 50  0000 C CNN
+F 1 "CMM-4737DT-26186-TR" H 7300 2076 50  0000 C CNN
+F 2 "My Libraries:XDCR_CMM-4737DT-26186-TR" H 6700 1000 50  0001 L BNN
+F 3 "" H 7300 1600 50  0001 L BNN
+F 4 "Unavailable" H 7100 900 50  0001 L BNN "Field4"
+F 5 "None" H 7300 1600 50  0001 L BNN "Field5"
+F 6 "CUI Inc." H 6700 900 50  0001 L BNN "Field6"
+F 7 "None" H 7300 1600 50  0001 L BNN "Field7"
+F 8 "CMM-4737DT-26186-TR" H 7600 900 50  0001 L BNN "Field8"
+	1    7300 1600
+	1    0    0    -1
+$EndComp
+Text Label 6200 1700 0    50   ~ 0
+PDM_CLK
+Text Label 6200 1500 0    50   ~ 0
+PDM_DATA
+Wire Wire Line
+	6200 1500 6600 1500
+Wire Wire Line
+	6200 1700 6600 1700
+$Comp
+L power:GND #PWR0108
+U 1 1 5ECDBE0F
+P 8100 1950
+F 0 "#PWR0108" H 8100 1700 50  0001 C CNN
+F 1 "GND" H 8105 1777 50  0000 C CNN
+F 2 "" H 8100 1950 50  0001 C CNN
+F 3 "" H 8100 1950 50  0001 C CNN
+	1    8100 1950
+	1    0    0    -1
+$EndComp
+Wire Wire Line
+	8000 1800 8100 1800
+Wire Wire Line
+	8100 1800 8100 1900
+Wire Wire Line
+	8000 1900 8100 1900
+Connection ~ 8100 1900
+Wire Wire Line
+	8100 1900 8100 1950
+Wire Wire Line
+	8000 1600 8100 1600
+Wire Wire Line
+	8100 1600 8100 1800
+Connection ~ 8100 1800
 $EndSCHEMATC

Commit message: Minor updates
Connections:
- net 32KHz: now also J2.5 (Pin_5); no longer J2.7 (Pin_7)
- net DS3231_INT: now also J2.4 (Pin_4); no longer J2.6 (Pin_6)
- net DS3231_RST: now also J2.3 (Pin_3); no longer J2.5 (Pin_5)
- net PDM_CLK: now also J2.6 (Pin_6); no longer J2.3 (Pin_3)
- net PDM_DATA: now also J2.7 (Pin_7); no longer J2.4 (Pin_4)
Other:
- note removed: "TODO: Battery measuring circuit"
Changed lines of the file:
@@
 Text Label 8550 1450 0    50   ~ 0
 SD-CS
+Text Label 10400 1950 2    50   ~ 0
+PDM_CLK
+Text Label 10400 1850 2    50   ~ 0
+PDM_DATA
 Text Label 10400 2250 2    50   ~ 0
-PDM_CLK
+DS3231_RST
 Text Label 10400 2150 2    50   ~ 0
-PDM_DATA
-Text Notes 8550 850  0    50   ~ 0
-TODO: Battery measuring circuit
+DS3231_INT
 Text Label 10400 2050 2    50   ~ 0
-DS3231_RST
-Text Label 10400 1950 2    50   ~ 0
-DS3231_INT
-Text Label 10400 1850 2    50   ~ 0
 32KHz
 Text Label 8550 1850 0    50   ~ 0

Commit message: Finished v1 layout
Thanks to everyone on the stream!
Connections:
- net SD-CD is gone; now on net SD_CD: J1.12 (Pin_12)
- net SD-CS is gone; now on net SD_CS: J1.11 (Pin_11)
- net Batt_Meas: now also J1.8 (Pin_8); no longer J1.9 (Pin_9)
- net Batt_Meas_En: now also J1.9 (Pin_9); no longer J2.8 (Pin_8)
- net SHT30-ALERT renamed SHT30_ALERT
- net SHT30_ALERT: now also J2.8 (Pin_8); no longer J1.8 (Pin_8)
Changed lines of the file:
@@
 	8550 2050 9100 2050
 Text Label 8550 1350 0    50   ~ 0
-SD-CD
+SD_CD
 $Comp
 L power:GND #PWR0131
@@
 	3700 6000 3950 6000
 Text Label 8550 1450 0    50   ~ 0
-SD-CS
+SD_CS
 Text Label 10400 1950 2    50   ~ 0
 PDM_CLK
@@
 Text Label 8550 1850 0    50   ~ 0
 APDS_INT
+Text Label 10400 1750 2    50   ~ 0
+SHT30_ALERT
 Text Label 8550 1750 0    50   ~ 0
-SHT30-ALERT
-Text Label 8550 1650 0    50   ~ 0
 Batt_Meas
 Text Label 8550 1550 0    50   ~ 0
@@
 Wire Wire Line
 	9250 5300 9400 5300
-Text Label 10400 1750 2    50   ~ 0
+Text Label 8550 1650 0    50   ~ 0
 Batt_Meas_En
 Wire Wire Line
@@
 	3500 2350 3500 2300
 Text Label 4050 3900 2    50   ~ 0
-SHT30-ALERT
+SHT30_ALERT
 $Comp
 L My_Library:CMM-4737DT-26186-TR U5
