File: hardware/Bald Sense Wing v3.kicad_sch (KiCad schematic)
At the start: 48 parts, among them J1 feather long, J2 feather short, J3 1140084168, J4 STEMMA-QT, Q1 Q_PNP_BEC, Q2 Q_NPN_BEC, SW1 Reset, U1 APDS-9960, U2 DS3231MZ, U3 SHT30-DIS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

Commit message: 14 unrouted
Parts:
- C7: now not fitted
- SW1: value Reset -> PTS810; footprint (none) -> Button_Switch_SMD:SW_SPST_PTS810; Function (none) -> Reset
- TP1, TP2, TP3, TP4, TP5, TP6, TP8: value TestPoint_Harwin -> Test Point; footprint My Libraries:Harwin-S1751-46-Test-Point -> TestPoint:TestPoint_Pad_1.0x1.0mm
- TP7: value TestPoint_Harwin -> FLG; footprint My Libraries:Harwin-S1751-46-Test-Point -> TestPoint:TestPoint_Pad_1.0x1.0mm
Connections:
- net +3.3V: now also J4.2 (Pin_2); no longer J4.3 (Pin_3)
- net GND: now also J4.1 (Pin_1); no longer J4.4 (Pin_4)
- net SCL: now also J4.4 (Pin_4); no longer J4.1 (Pin_1)
- net SDA: now also J4.3 (Pin_3); no longer J4.2 (Pin_2)
Other:
- moved on the sheet: SW1
Changed lines of the file:
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@@
 	(wire
 		(pts
-			(xy 179.07 21.59) (xy 173.99 21.59)
+			(xy 179.07 25.4) (xy 173.99 25.4)
 		)
 		(stroke
@@
 	)
 	(label "~{RST}"
-		(at 179.07 21.59 180)
+		(at 179.07 25.4 180)
 		(fields_autoplaced yes)
 		(effects
@@
 		(in_bom yes)
 		(on_board yes)
-		(dnp no)
+		(dnp yes)
 		(property "Reference" "C7"
 			(at 110.2868 153.7716 0)
@@
 	(symbol
 		(lib_id "power:GND")
-		(at 163.83 21.59 0)
+		(at 163.83 25.4 0)
 		(unit 1)
 		(exclude_from_sim no)
@@
 		(dnp no)
 		(property "Reference" "#PWR019"
-			(at 163.83 27.94 0)
+			(at 163.83 31.75 0)
 			(effects
 				(font
@@
 		)
 		(property "Value" "GND"
-			(at 163.957 25.9842 0)
+			(at 163.957 29.7942 0)
 			(effects
 				(font
@@
 		)
 		(property "Footprint" ""
-			(at 163.83 21.59 0)
+			(at 163.83 25.4 0)
 			(effects
 				(font
@@
 		)
 		(property "Datasheet" ""
-			(at 163.83 21.59 0)
+			(at 163.83 25.4 0)
 			(effects
 				(font
@@
 		)
 		(property "Description" ""
-			(at 163.83 21.59 0)
+			(at 163.83 25.4 0)
 			(effects
 				(font
@@
 			)
 		)
-		(property "Value" "TestPoint_Harwin"
+		(property "Value" "Test Point"
 			(at 201.93 53.34 0)
 			(effects
@@
 			)
 		)
-		(property "Footprint" "My Libraries:Harwin-S1751-46-Test-Point"
+		(property "Footprint" "TestPoint:TestPoint_Pad_1.0x1.0mm"
 			(at 207.01 48.26 0)
 			(effects
@@
 			)
 		)
-		(property "Value" "TestPoint_Harwin"
+		(property "Value" "FLG"
 			(at 204.47 107.95 0)
 			(effects
@@
 			)
 		)
-		(property "Footprint" "My Libraries:Harwin-S1751-46-Test-Point"
+		(property "Footprint" "TestPoint:TestPoint_Pad_1.0x1.0mm"
 			(at 199.39 113.03 0)
 			(effects
@@
 			)
 		)
-		(property "Value" "TestPoint_Harwin"
+		(property "Value" "Test Point"
 			(at 236.22 106.68 0)
 			(effects
@@
 			)
 		)
-		(property "Footprint" "My Libraries:Harwin-S1751-46-Test-Point"
+		(property "Footprint" "TestPoint:TestPoint_Pad_1.0x1.0mm"
 			(at 241.3 101.6 0)
 			(effects
@@
 	(symbol
 		(lib_id "Connector_Generic:Conn_01x04")
-		(at 214.63 83.82 0)
+		(at 214.63 86.36 0)
+		(mirror x)
 		(unit 1)
 		(exclude_from_sim no)
@@
 		(on_board yes)
 		(dnp no)
-		(fields_autoplaced yes)
 		(property "Reference" "J4"
-			(at 217.17 82.5499 0)
+			(at 217.17 87.6301 0)
 			(effects
 				(font
@@
 		)
 		(property "Value" "STEMMA-QT"
-			(at 217.17 85.0899 0)
+			(at 217.17 85.0901 0)
 			(effects
 				(font
@@
 		)
 		(property "Footprint" "Connector_JST:JST_SH_BM04B-SRSS-TB_1x04-1MP_P1.00mm_Vertical"
-			(at 214.63 83.82 0)
+			(at 214.63 86.36 0)
 			(effects
 				(font
@@
 		)
 		(property "Datasheet" "~"
-			(at 214.63 83.82 0)
+			(at 214.63 86.36 0)
 			(effects
 				(font
@@
 		)
 		(property "Description" "Generic connector, single row, 01x04, script generated (kicad-library-utils/schlib/autogen/connector/)"
-			(at 214.63 83.82 0)
+			(at 214.63 86.36 0)
 			(effects
 				(font
@@
 		)
 		(property "Field5" "JST SH"
-			(at 217.17 87.6299 0)
+			(at 217.17 82.5501 0)
 			(effects
 				(font
@@
 			)
 		)
-		(property "Value" "TestPoint_Harwin"
+		(property "Value" "Test Point"
 			(at 246.38 149.86 0)
 			(effects
@@
 			)
 		)
-		(property "Footprint" "My Libraries:Harwin-S1751-46-Test-Point"
+		(property "Footprint" "TestPoint:TestPoint_Pad_1.0x1.0mm"
 			(at 251.46 144.78 0)
 			(effects
@@
 			)
 		)
-		(property "Value" "TestPoint_Harwin"
+		(property "Value" "Test Point"
 			(at 201.93 55.88 0)
 			(effects
@@
 			)
 		)
-		(property "Footprint" "My Libraries:Harwin-S1751-46-Test-Point"
+		(property "Footprint" "TestPoint:TestPoint_Pad_1.0x1.0mm"
 			(at 207.01 50.8 0)
 			(effects
@@
 	(symbol
 		(lib_id "Switch:SW_SPST")
-		(at 168.91 21.59 0)
+		(at 168.91 25.4 0)
 		(unit 1)
 		(exclude_from_sim no)
@@
 		(fields_autoplaced yes)
 		(property "Reference" "SW1"
-			(at 168.91 15.24 0)
+			(at 168.91 16.51 0)
 			(effects
 				(font
@@
 			)
 		)
-		(property "Value" "Reset"
-			(at 168.91 17.78 0)
+		(property "Value" "PTS810"
+			(at 168.91 19.05 0)
 			(effects
 				(font
@@
 			)
 		)
-		(property "Footprint" ""
-			(at 168.91 21.59 0)
+		(property "Footprint" "Button_Switch_SMD:SW_SPST_PTS810"
+			(at 168.91 25.4 0)
 			(effects
 				(font
@@
 		)
 		(property "Datasheet" "~"
-			(at 168.91 21.59 0)
+			(at 168.91 25.4 0)
 			(effects
 				(font
@@
 		)
 		(property "Description" "Single Pole Single Throw (SPST) switch"
-			(at 168.91 21.59 0)
+			(at 168.91 25.4 0)
 			(effects
 				(font
@@
 			)
 		)
+		(property "Function" "Reset"
+			(at 168.91 21.59 0)
+			(effects
+				(font
+					(size 1.27 1.27)
+				)
+			)
+		)
 		(pin "2"
 		)
@@
 			)
 		)
-		(property "Value" "TestPoint_Harwin"
+		(property "Value" "Test Point"
 			(at 241.3 33.02 0)
 			(effects
@@
 			)
 		)
-		(property "Footprint" "My Libraries:Harwin-S1751-46-Test-Point"
+		(property "Footprint" "TestPoint:TestPoint_Pad_1.0x1.0mm"
 			(at 236.22 38.1 0)
 			(effects
@@
 			)
 		)
-		(property "Value" "TestPoint_Harwin"
+		(property "Value" "Test Point"
 			(at 201.93 58.42 0)
 			(effects
@@
 			)
 		)
-		(property "Footprint" "My Libraries:Harwin-S1751-46-Test-Point"
+		(property "Footprint" "TestPoint:TestPoint_Pad_1.0x1.0mm"
 			(at 207.01 53.34 0)
 			(effects
@@
 			)
 		)
-		(property "Value" "TestPoint_Harwin"
+		(property "Value" "Test Point"
 			(at 201.93 25.4 0)
 			(effects
@@
 			)
 		)
-		(property "Footprint" "My Libraries:Harwin-S1751-46-Test-Point"
+		(property "Footprint" "TestPoint:TestPoint_Pad_1.0x1.0mm"
 			(at 207.01 20.32 0)
 			(effects
